Commit message: Fix urdf not showing in simulation and rviz

File: roverrobotics_description/urdf/indoor_miti_payload.urdf (robot description, URDF)
Before this commit: robot rover_miti_payload, 1 links, 1 joints
Links:
- link payload_link: geometry collision mesh filename=file://$(find roverrobotics_description)/meshes/rover_paylo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; visual mesh filename=file://$(find roverrobotics_description)/meshes/rover_paylo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

File: roverrobotics_description/urdf/mini.urdf (robot description, URDF)
Before this commit: robot rover_mini, 6 links, 5 joints
Links:
- link chassis_link: geometry collision mesh filename=file://$(find roverrobotics_description)/meshes/mini_chassi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; visual mesh filename=file://$(find roverrobotics_description)/meshes/mini_chassi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
- link fl_wheel_link: geometry collision mesh filename=file://$(find roverrobotics_description)/meshes/hub_6.5in.d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; visual mesh filename=file://$(find roverrobotics_description)/meshes/hub_6.5in.d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
- link fr_wheel_link: geometry collision mesh filename=file://$(find roverrobotics_description)/meshes/hub_6.5in.d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; visual mesh filename=file://$(find roverrobotics_description)/meshes/hub_6.5in.d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
- link rl_wheel_link: geometry collision mesh filename=file://$(find roverrobotics_description)/meshes/hub_6.5in.d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; visual mesh filename=file://$(find roverrobotics_description)/meshes/hub_6.5in.d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
- link rr_wheel_link: geometry collision mesh filename=file://$(find roverrobotics_description)/meshes/hub_6.5in.d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; visual mesh filename=file://$(find roverrobotics_description)/meshes/hub_6.5in.d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

File: roverrobotics_description/urdf/mini_payload.urdf (robot description, URDF)
Before this commit: robot rover_mini_payload, 1 links, 1 joints
Links:
- link payload_link: geometry collision mesh filename=file://$(find roverrobotics_description)/meshes/rover_paylo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; visual mesh filename=file://$(find roverrobotics_description)/meshes/rover_paylo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

File: roverrobotics_description/urdf/miti.urdf (robot description, URDF)
Before this commit: robot rover_miti, 6 links, 5 joints
Links:
- link chassis_link: geometry collision mesh filename=file://$(find roverrobotics_description)/meshes/miti_chassi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; visual mesh filename=file://$(find roverrobotics_description)/meshes/miti_chassi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
- link fl_wheel_link: geometry collision mesh filename=file://$(find roverrobotics_description)/meshes/hub_10in.dae; visual mesh filename=file://$(find roverrobotics_description)/meshes/hub_10in.dae
- link fr_wheel_link: geometry collision mesh filename=file://$(find roverrobotics_description)/meshes/hub_10in.dae; visual mesh filename=file://$(find roverrobotics_description)/meshes/hub_10in.dae
- link rl_wheel_link: geometry collision mesh filename=file://$(find roverrobotics_description)/meshes/hub_10in.dae; visual mesh filename=file://$(find roverrobotics_description)/meshes/hub_10in.dae
- link rr_wheel_link: geometry collision mesh filename=file://$(find roverrobotics_description)/meshes/hub_10in.dae; visual mesh filename=file://$(find roverrobotics_description)/meshes/hub_10in.dae

File: roverrobotics_description/urdf/miti_payload.urdf (robot description, URDF)
Before this commit: robot rover_miti_payload, 1 links, 1 joints
Links:
- link payload_link: geometry collision mesh filename=file://$(find roverrobotics_description)/meshes/rover_paylo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; visual mesh filename=file://$(find roverrobotics_description)/meshes/rover_paylo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
