Commit message: wheels should spin

File: roverrobotics_description/urdf/indoor_miti.urdf (robot description, URDF)
Before this commit: robot rover_miti, 6 links, 5 joints
Joints:
- joint fl_wheel_to_chassis: axis (none) -> 0 1 0; origin (none) -> xyz=0 0 0; type fixed -> continuous
- joint fr_wheel_to_chassis: axis (none) -> 0 1 0; origin (none) -> xyz=0 0 0; type fixed -> continuous
- joint rl_wheel_to_chassis: axis (none) -> 0 1 0; origin (none) -> xyz=0 0 0; type fixed -> continuous
- joint rr_wheel_to_chassis: axis (none) -> 0 1 0; origin (none) -> xyz=0 0 0; type fixed -> continuous

File: roverrobotics_description/urdf/mini.urdf (robot description, URDF)
Before this commit: robot rover_mini, 6 links, 5 joints
Joints:
- joint fl_wheel_to_chassis: axis (none) -> 0 1 0; origin (none) -> xyz=0 0 0; type fixed -> continuous
- joint fr_wheel_to_chassis: axis (none) -> 0 1 0; origin (none) -> xyz=0 0 0; type fixed -> continuous
- joint rl_wheel_to_chassis: axis (none) -> 0 1 0; origin (none) -> xyz=0 0 0; type fixed -> continuous
- joint rr_wheel_to_chassis: axis (none) -> 0 1 0; origin (none) -> xyz=0 0 0; type fixed -> continuous

File: roverrobotics_description/urdf/miti.urdf (robot description, URDF)
Before this commit: robot rover_miti, 6 links, 5 joints
Joints:
- joint fl_wheel_to_chassis: axis (none) -> 0 1 0; origin (none) -> xyz=0 0 0; type fixed -> continuous
- joint fr_wheel_to_chassis: axis (none) -> 0 1 0; origin (none) -> xyz=0 0 0; type fixed -> continuous
- joint rl_wheel_to_chassis: axis (none) -> 0 1 0; origin (none) -> xyz=0 0 0; type fixed -> continuous
- joint rr_wheel_to_chassis: axis (none) -> 0 1 0; origin (none) -> xyz=0 0 0; type fixed -> continuous

Commit message: Fix joint positioning for wheels

File: roverrobotics_description/urdf/indoor_miti.urdf (robot description, URDF)
Before this commit: robot rover_miti, 6 links, 5 joints
Joints:
- joint fl_wheel_to_chassis: origin xyz=0 0 0 -> xyz=${wheel_x_offset} ${wheel_y_offset} ${wheel_z_offset}
- joint fr_wheel_to_chassis: origin xyz=0 0 0 -> xyz=${wheel_x_offset} ${-wheel_y_offset} ${wheel_z_offset}
- joint rl_wheel_to_chassis: origin xyz=0 0 0 -> xyz=${-wheel_x_offset} ${wheel_y_offset} ${wheel_z_offset}
- joint rr_wheel_to_chassis: origin xyz=0 0 0 -> xyz=${-wheel_x_offset} ${-wheel_y_offset} ${wheel_z_offset}

File: roverrobotics_description/urdf/mini.urdf (robot description, URDF)
Before this commit: robot rover_mini, 6 links, 5 joints
Joints:
- joint fl_wheel_to_chassis: origin xyz=0 0 0 -> xyz=${wheel_x_offset - front_wheel_x_offset} ${wheel_y_offset} ${wheel_z_offset}
- joint fr_wheel_to_chassis: origin xyz=0 0 0 -> xyz=${wheel_x_offset - front_wheel_x_offset}  ${-wheel_y_offset} ${wheel_z_offset}
- joint rl_wheel_to_chassis: origin xyz=0 0 0 -> xyz=${-wheel_x_offset} ${wheel_y_offset} ${wheel_z_offset}
- joint rr_wheel_to_chassis: origin xyz=0 0 0 -> xyz=${-wheel_x_offset} ${-wheel_y_offset} ${wheel_z_offset}

File: roverrobotics_description/urdf/miti.urdf (robot description, URDF)
Before this commit: robot rover_miti, 6 links, 5 joints
Joints:
- joint fl_wheel_to_chassis: origin xyz=0 0 0 -> xyz=${wheel_x_offset} ${wheel_y_offset} ${wheel_z_offset}
- joint fr_wheel_to_chassis: origin xyz=0 0 0 -> xyz=${wheel_x_offset} ${-wheel_y_offset} ${wheel_z_offset}
- joint rl_wheel_to_chassis: origin xyz=0 0 0 -> xyz=${-wheel_x_offset} ${wheel_y_offset} ${wheel_z_offset}
- joint rr_wheel_to_chassis: origin xyz=0 0 0 -> xyz=${-wheel_x_offset} ${-wheel_y_offset} ${wheel_z_offset}

Commit message: Add basic simulation setup

File: roverrobotics_description/urdf/indoor_miti.urdf (robot description, URDF)
Before this commit: robot rover_miti, 6 links, 5 joints
Links:
- link chassis_link: geometry collision mesh filename=file://$(find roverrobotics_description)/meshes/miti_chassi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; visual mesh filename=file://$(find roverrobotics_description)/meshes/miti_chassi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
- link fl_wheel_link: geometry collision mesh filename=file://$(find roverrobotics_description)/meshes/hub_6.5in.d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; visual mesh filename=file://$(find roverrobotics_description)/meshes/hub_6.5in.d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
- link fr_wheel_link: geometry collision mesh filename=file://$(find roverrobotics_description)/meshes/hub_6.5in.d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; visual mesh filename=file://$(find roverrobotics_description)/meshes/hub_6.5in.d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
- link rl_wheel_link: geometry collision mesh filename=file://$(find roverrobotics_description)/meshes/hub_6.5in.d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; visual mesh filename=file://$(find roverrobotics_description)/meshes/hub_6.5in.d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
- link rr_wheel_link: geometry collision mesh filename=file://$(find roverrobotics_description)/meshes/hub_6.5in.d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; visual mesh filename=file://$(find roverrobotics_description)/meshes/hub_6.5in.d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

Commit message: Fix chassis_link frame positioning

File: roverrobotics_description/urdf/indoor_miti.urdf (robot description, URDF)
Before this commit: robot rover_miti, 6 links, 5 joints
Joints:
- joint base_to_chassis: origin (none) -> xyz=0 0 0.061

File: roverrobotics_description/urdf/indoor_miti_payload.urdf (robot description, URDF)
Before this commit: robot rover_miti_payload, 1 links, 1 joints
Joints:
- joint payload_to_chassis: origin (none) -> xyz=0 0 0.1645

File: roverrobotics_description/urdf/mini.urdf (robot description, URDF)
Before this commit: robot rover_mini, 6 links, 5 joints
Joints:
- joint base_to_chassis: origin (none) -> xyz=0 0 0.0965

File: roverrobotics_description/urdf/mini_payload.urdf (robot description, URDF)
Before this commit: robot rover_mini_payload, 1 links, 1 joints
Joints:
- joint payload_to_chassis: origin (none) -> xyz=0 0 0.1105

File: roverrobotics_description/urdf/miti.urdf (robot description, URDF)
Before this commit: robot rover_miti, 6 links, 5 joints
Joints:
- joint base_to_chassis: origin (none) -> xyz=0 0 0.104

File: roverrobotics_description/urdf/miti_payload.urdf (robot description, URDF)
Before this commit: robot rover_miti_payload, 1 links, 1 joints
Joints:
- joint payload_to_chassis: origin (none) -> xyz=0 0.0115 0.156 rpy=0 0 0
