Commit message: Finish inertial values for 2wd rover

File: roverrobotics_description/urdf/rover_2wd.urdf (robot description, URDF)
Before this commit: robot rover_2wd, 8 links, 7 joints
Links:
- link rl_castor_housing_link: mass ${wheel_mass} -> ${castor_housing_mass}
- link rl_castor_link: mass ${wheel_mass} -> ${castor_mass}
- link rr_castor_housing_link: mass ${wheel_mass} -> ${castor_housing_mass}
- link rr_castor_link: mass ${wheel_mass} -> ${castor_mass}
