Commit message: Create URDF models for rover mini and miti

File: roverrobotics_description/urdf/mini.urdf (robot description, URDF)
Before this commit: robot onshape, 1 links, 0 joints
Links:
- added link chassis_link, mass ${chassis_mass}; collision mesh filename=package://roverrobotics_description/meshes/mini_chassis.dae; visual mesh filename=package://roverrobotics_description/meshes/mini_chassis.dae
- added link fl_wheel_link, mass ${wheel_mass}; collision mesh filename=package://roverrobotics_description/meshes/hub_6.5in.dae; visual mesh filename=package://roverrobotics_description/meshes/hub_6.5in.dae
- added link fr_wheel_link, mass ${wheel_mass}; collision mesh filename=package://roverrobotics_description/meshes/hub_6.5in.dae; visual mesh filename=package://roverrobotics_description/meshes/hub_6.5in.dae
- added link rl_wheel_link, mass ${wheel_mass}; collision mesh filename=package://roverrobotics_description/meshes/hub_6.5in.dae; visual mesh filename=package://roverrobotics_description/meshes/hub_6.5in.dae
- added link rr_wheel_link, mass ${wheel_mass}; collision mesh filename=package://roverrobotics_description/meshes/hub_6.5in.dae; visual mesh filename=package://roverrobotics_description/meshes/hub_6.5in.dae
- link base_link: mass 8 -> None; geometry 
Joints:
- added joint base_to_chassis: type fixed, parent base_link, child chassis_link
- added joint fl_wheel_to_chassis: type fixed, parent chassis_link, child fl_wheel_link
- added joint fr_wheel_to_chassis: type fixed, parent chassis_link, child fr_wheel_link
- added joint rl_wheel_to_chassis: type fixed, parent chassis_link, child rl_wheel_link
- added joint rr_wheel_to_chassis: type fixed, parent chassis_link, child rr_wheel_link

File: roverrobotics_description/urdf/miti.urdf (robot description, URDF)
Before this commit: robot onshape, 1 links, 0 joints
Links:
- added link chassis_link, mass ${chassis_mass}; collision mesh filename=package://roverrobotics_description/meshes/miti_chassis.dae; visual mesh filename=package://roverrobotics_description/meshes/miti_chassis.dae
- added link fl_wheel_link, mass ${wheel_mass}; collision mesh filename=package://roverrobotics_description/meshes/hub_10in.dae; visual mesh filename=package://roverrobotics_description/meshes/hub_10in.dae
- added link fr_wheel_link, mass ${wheel_mass}; collision mesh filename=package://roverrobotics_description/meshes/hub_10in.dae; visual mesh filename=package://roverrobotics_description/meshes/hub_10in.dae
- added link rl_wheel_link, mass ${wheel_mass}; collision mesh filename=package://roverrobotics_description/meshes/hub_10in.dae; visual mesh filename=package://roverrobotics_description/meshes/hub_10in.dae
- added link rr_wheel_link, mass ${wheel_mass}; collision mesh filename=package://roverrobotics_description/meshes/hub_10in.dae; visual mesh filename=package://roverrobotics_description/meshes/hub_10in.dae
- link base_link: mass 20 -> None; geometry 
Joints:
- added joint base_to_chassis: type fixed, parent base_link, child chassis_link
- added joint fl_wheel_to_chassis: type fixed, parent chassis_link, child fl_wheel_link
- added joint fr_wheel_to_chassis: type fixed, parent chassis_link, child fr_wheel_link
- added joint rl_wheel_to_chassis: type fixed, parent chassis_link, child rl_wheel_link
- added joint rr_wheel_to_chassis: type fixed, parent chassis_link, child rr_wheel_link

Commit message: updated URDFs

File: roverrobotics_description/urdf/mini.urdf (robot description, URDF)
Before this commit: robot rover_mini, 6 links, 5 joints
Links:
- link fl_wheel_link: geometry collision mesh filename=file://$(find roverrobotics_description)/meshes/65wheels.dae; visual mesh filename=file://$(find roverrobotics_description)/meshes/65wheels.dae
- link fr_wheel_link: geometry collision mesh filename=file://$(find roverrobotics_description)/meshes/65wheels.dae; visual mesh filename=file://$(find roverrobotics_description)/meshes/65wheels.dae
- link rl_wheel_link: geometry collision mesh filename=file://$(find roverrobotics_description)/meshes/65wheels.dae; visual mesh filename=file://$(find roverrobotics_description)/meshes/65wheels.dae
- link rr_wheel_link: geometry collision mesh filename=file://$(find roverrobotics_description)/meshes/65wheels.dae; visual mesh filename=file://$(find roverrobotics_description)/meshes/65wheels.dae
Joints:
- joint base_to_chassis: origin xyz=0 0 0.0965 -> xyz=0 0 0.061
- joint fl_wheel_to_chassis: origin xyz=${wheel_x_offset - front_wheel_x_offset} ${wheel_y_offset} ${wheel_z_offset} -> xyz=${wheel_x_offset} ${wheel_y_offset} ${wheel_z_offset}
- joint fr_wheel_to_chassis: origin xyz=${wheel_x_offset - front_wheel_x_offset}  ${-wheel_y_offset} ${wheel_z_offset} -> xyz=${wheel_x_offset} ${-wheel_y_offset} ${wheel_z_offset}
