Commit message: Consolidate payload into one file

File: roverrobotics_description/urdf/accessories/rover_dev_payload.urdf (robot description, URDF)
Before this commit: robot rover_mini_payload, 1 links, 1 joints
Joints:
- joint payload_to_chassis: origin xyz=0 0 0.1105 -> xyz=0 0 ${payload_z_offset}

Commit message: Flipper urdf with inertia

File: roverrobotics_description/urdf/accessories/rover_dev_payload.urdf (robot description, URDF)
Before this commit: robot rover_miti_payload, 1 links, 1 joints
Links:
- link payload_link: mass None -> 2.95

File: roverrobotics_description/urdf/flipper.urdf (robot description, URDF)
Before this commit: robot rover_miti, 8 links, 7 joints
Links:
- link left_track_link: mass ${wheel_mass} -> None
- link right_track_link: mass ${wheel_mass} -> None
