Commit message: Rotate rplidar 180 degrees for physical model

File: roverrobotics_description/urdf/accessories/rplidar_s2.urdf (robot description, URDF)
Before this commit: robot rplidar_s2, 1 links, 1 joints
Joints:
- joint lidar_to_payload: origin xyz=0.174 0 0.10 rpy=0 0 0 -> xyz=0.174 0 0.10 rpy=0 0 3.1415
