Commit message: updated gps.urdf

File: roverrobotics_description/urdf/accessories/gps.urdf (robot description, URDF)
Before this commit: robot None, 0 links, 0 joints
Links:
- added link gps_link
Joints:
- added joint gps_to_payload: type fixed, parent payload_link, child gps_link, origin xyz=-0.10 0.05 0.135 rpy=0 0 0
